Commit message: upper arm joint renamed

File: urdf/two_link.urdf (robot description, URDF)
Before this commit: robot two_link, 4 links, 3 joints
Joints:
- removed joint base_to_upper_arm
- added joint base_to_upper: type continuous, parent base_link, child upper_arm, origin xyz=0.0 0 0, axis 0 1 0
