Commit message: urdf updated to have all 4 limbs and transform tested as well.

File: urdf/upper_body.urdf (robot description, URDF)
Before this commit: robot two_link, 7 links, 6 joints
Links:
- added link head; visual sphere radius=0.06
- added link left_arm; visual cylinder length=0.25 radius=0.03
- added link left_elbow; visual sphere radius=0.01
- added link left_foot; visual sphere radius=0.03
- added link left_forearm; visual cylinder length=0.2 radius=0.03
- added link left_hand; visual sphere radius=0.03
- added link left_hip; visual sphere radius=0.01
- added link left_knee; visual sphere radius=0.01
- added link left_shin; visual cylinder length=0.2 radius=0.03
- added link left_shoulder; visual sphere radius=0.01
- added link left_thigh; visual cylinder length=0.3 radius=0.05
- added link right_foot; visual sphere radius=0.03
- added link right_hip; visual sphere radius=0.01
- added link right_knee; visual sphere radius=0.01
- added link right_shin; visual cylinder length=0.2 radius=0.03
- added link right_thigh; visual cylinder length=0.3 radius=0.05
Joints:
- added joint left_ankle: type fixed, parent left_shin, child left_foot, origin xyz=0.1 0 0, axis 0 0 1
- added joint left_arm_to_elbow: type revolute, parent left_arm, child left_elbow, origin xyz=0.125 0 0, limit lower=0 upper=2.5 effort=10.0 velocity=5.0
- added joint left_elbow_to_lower: type fixed, parent left_elbow, child left_forearm, origin xyz=0.1 0 0, axis 0 0 1
- added joint left_hip: type continuous, parent body, child left_hip, origin xyz=0.0 0.075 -0.5, axis 0 0 1
- added joint left_hip_to_thigh: type fixed, parent left_hip, child left_thigh, origin xyz=0.125 0 0, axis 0 0 1
- added joint left_knee_to_shin: type fixed, parent left_knee, child left_shin, origin xyz=0.1 0 0, axis 0 0 1
- added joint left_shoulder: type continuous, parent body, child left_shoulder, origin xyz=0.0 0.15 0, axis 0 0 1
- added joint left_shoulder_to_upper: type fixed, parent left_shoulder, child left_arm, origin xyz=0.125 0 0, axis 0 0 1
- added joint left_thigh_to_knee: type revolute, parent left_thigh, child left_knee, origin xyz=0.15 0 0, limit lower=0 upper=2.5 effort=10.0 velocity=5.0
- added joint left_wrist: type fixed, parent left_forearm, child left_hand, origin xyz=0.1 0 0, axis 0 0 1
- added joint neck: type fixed, parent body, child head, origin xyz=0 0 0.1, axis 0 0 1
- added joint right_ankle: type fixed, parent right_shin, child right_foot, origin xyz=0.1 0 0, axis 0 0 1
- added joint right_hip: type continuous, parent body, child right_hip, origin xyz=0.0 -0.075 -0.5, axis 0 0 1
- added joint right_hip_to_thigh: type fixed, parent right_hip, child right_thigh, origin xyz=0.125 0 0, axis 0 0 1
- added joint right_knee_to_shin: type fixed, parent right_knee, child right_shin, origin xyz=0.1 0 0, axis 0 0 1
- added joint right_thigh_to_knee: type revolute, parent right_thigh, child right_knee, origin xyz=0.15 0 0, limit lower=0 upper=2.5 effort=10.0 velocity=5.0
- joint right_arm_to_elbow: origin xyz=-0.1 0 0 -> xyz=0.125 0 0
